Commit message: Robot with speed and direction using RViz, ROS, URDF, Xacro etc

File: src/project_one/urdf/robot_base.urdf.xacro (robot description, xacro)
@@ -17,10 +17,5 @@
     <color rgba="1 1 1 1"/>
   </material>
-  <xacro:macro name="default_inertial" params="mass">
-    <inertial>
-      <mass value="${mass}" />
-      <inertia ixx="1.0" ixy="0.0" ixz="0.0" iyy="1.0" iyz="0.0" izz="1.0" />
-    </inertial>
-  </xacro:macro>
+  <xacro:include filename="$(find project_one)/urdf/robot_inertial_essentials.xacro" />
   <link name="base_link">
     <visual>
@@ -37,7 +32,9 @@
     <xacro:default_inertial mass="10"/>
   </link>
-	<xacro:include filename="$(find project_one)/urdf/robot_essentials.xacro" />
-	<xacro:robot_wheel prefix="right" originY="-0.22" />
-	<xacro:robot_wheel prefix="left" originY="0.22"/>
+  <xacro:include filename="$(find project_one)/urdf/robot_essentials.xacro" />
+<!--	<xacro:robot_wheel prefix="right" originY="-0.22" />
+	<xacro:robot_wheel prefix="left" originY="0.22"/> -->
+  <xacro:leg prefix="right" reflect="-1" />
+  <xacro:leg prefix="left" reflect="1" />
   <joint name="gripper_extension" type="prismatic">
     <parent link="base_link"/>
@@ -45,4 +42,6 @@
     <limit effort="1000.0" lower="-${width*2-.02}" upper="0" velocity="0.5"/>
     <origin rpy="0 0 0" xyz="${width-.01} 0 0.2"/>
+    <limit effort="30" velocity="0.2"/>
+    <dynamics damping="0.0" friction="0.0"/>
   </joint>
   <link name="gripper_pole">
@@ -61,47 +60,14 @@
     <xacro:default_inertial mass="0.05"/>
   </link>
-  <xacro:macro name="gripper" params="prefix reflect">
-    <joint name="${prefix}_gripper_joint" type="revolute">
-      <axis xyz="0 0 ${reflect}"/>
-      <limit effort="1000.0" lower="0.0" upper="0.548" velocity="0.5"/>
-      <origin rpy="0 0 0" xyz="${polelen} ${reflect*0.01} 0"/>
-      <parent link="gripper_pole"/>
-      <child link="${prefix}_gripper"/>
+  <transmission name="gripper_extension_trans">
+    <type>transmission_interface/SimpleTransmission</type>
+    <actuator name="gripper_extension_motor">
+      <mechanicalReduction>1</mechanicalReduction>
+    </actuator>
+    <joint name="gripper_extension">
+      <hardwareInterface>PositionJointInterface</hardwareInterface>
     </joint>
-    <link name="${prefix}_gripper">
-      <visual>
-        <origin rpy="${(reflect-1)/2*pi} 0 0" xyz="0 0 0"/>
-        <geometry>
-          <mesh filename="package://urdf_tutorial/meshes/l_finger.dae"/>
-        </geometry>
-      </visual>
-      <collision>
-        <geometry>
-          <mesh filename="package://urdf_tutorial/meshes/l_finger.dae"/>
-        </geometry>
-        <origin rpy="${(reflect-1)/2*pi} 0 0" xyz="0 0 0"/>
-      </collision>
-      <xacro:default_inertial mass="0.05"/>
-    </link>
-    <joint name="${prefix}_tip_joint" type="fixed">
-      <parent link="${prefix}_gripper"/>
-      <child link="${prefix}_tip"/>
-    </joint>
-    <link name="${prefix}_tip">
-      <visual>
-        <origin rpy="${(reflect-1)/2*pi} 0 0" xyz="0.09137 0.00495 0"/>
-        <geometry>
-          <mesh filename="package://urdf_tutorial/meshes/l_finger_tip.dae"/>
-        </geometry>
-      </visual>
-      <collision>
-        <geometry>
-          <mesh filename="package://urdf_tutorial/meshes/l_finger_tip.dae"/>
-        </geometry>
-        <origin rpy="${(reflect-1)/2*pi} 0 0" xyz="0.09137 0.00495 0"/>
-      </collision>
-      <xacro:default_inertial mass="0.05"/>
-    </link>
-  </xacro:macro>
+  </transmission>
+  <xacro:include filename="$(find project_one)/urdf/robot_gripper.xacro" />
   <xacro:gripper prefix="left" reflect="1" />
   <xacro:gripper prefix="right" reflect="-1" />
@@ -125,5 +91,17 @@
     <axis xyz="0 0 1"/>
     <origin xyz="0 0 ${bodylen/2}"/>
+    <limit effort="30" velocity="1.0"/>
+    <dynamics damping="0.0" friction="0.0"/>
   </joint>
+  <!-- This block connects the head_swivel joint to an actuator (motor), which informs both simulation and visualization of the robot -->
+  <transmission name="head_swivel_trans">
+    <type>transmission_interface/SimpleTransmission</type>
+    <actuator name="$head_swivel_motor">
+      <mechanicalReduction>1</mechanicalReduction>
+    </actuator>
+    <joint name="head_swivel">
+      <hardwareInterface>PositionJointInterface</hardwareInterface>
+    </joint>
+  </transmission>
   <link name="box">
     <visual>
@@ -146,9 +124,9 @@
     <origin xyz="${.707*width+0.04} 0 ${.707*width}"/>
   </joint>
-<!--
+  <!-- Gazebo plugin for ROS Control -->
   <gazebo>
     <plugin name="gazebo_ros_control" filename="libgazebo_ros_control.so">
       <robotNamespace>/</robotNamespace>
     </plugin>
-  </gazebo>	 -->
+  </gazebo>
 </robot>

File: src/project_one/urdf/robot_essentials.xacro (robot description, xacro)
@@ -1,4 +1,89 @@
 <?xml version="1.0"?>
 <robot xmlns:xacro="http://ros.org/wiki/xacro" name="robot_essentials">
+	<xacro:macro name="wheel" params="prefix suffix reflect">
+		<link name="${prefix}_${suffix}_wheel">
+		  <visual>
+		    <origin xyz="0 0 0" rpy="${pi/2} 0 0" />
+		    <geometry>
+		      <cylinder radius="${wheeldiam/2}" length="0.1"/>
+		    </geometry>
+		    <material name="black"/>
+		  </visual>
+		  <collision>
+		    <origin xyz="0 0 0" rpy="${pi/2} 0 0" />
+		    <geometry>
+		      <cylinder radius="${wheeldiam/2}" length="0.1"/>
+		    </geometry>
+		  </collision>
+		  <xacro:default_inertial mass="1"/>
+		</link>
+		<joint name="${prefix}_${suffix}_wheel_joint" type="continuous">
+		  <axis xyz="0 1 0" rpy="0 0 0" />
+		  <parent link="${prefix}_base"/>
+		  <child link="${prefix}_${suffix}_wheel"/>
+		  <origin xyz="${baselen*reflect/3} 0 -${wheeldiam/2+.05}" rpy="0 0 0"/>
+		</joint>
+		<transmission name="${prefix}_${suffix}_wheel_trans">
+		  <type>transmission_interface/SimpleTransmission</type>
+		  <actuator name="${prefix}_${suffix}_wheel_motor">
+		    <mechanicalReduction>1</mechanicalReduction>
+		  </actuator>
+		  <joint name="${prefix}_${suffix}_wheel_joint">
+		    <hardwareInterface>VelocityJointInterface</hardwareInterface>
+		  </joint>
+		</transmission>
+		<gazebo reference="${prefix}_${suffix}_wheel">
+		  <mu1 value="200.0"/>
+		  <mu2 value="100.0"/>
+		  <kp value="10000000.0" />
+		  <kd value="1.0" />
+		  <material>Gazebo/Grey</material>
+		</gazebo>
+	  </xacro:macro>
+	  <xacro:macro name="leg" params="prefix reflect">
+		<link name="${prefix}_leg">
+		  <visual>
+		    <geometry>
+		      <box size="${leglen} 0.1 0.2"/>
+		    </geometry>
+		    <origin xyz="0 0 -${leglen/2}" rpy="0 ${pi/2} 0"/>
+		    <material name="white"/>
+		  </visual>
+		  <collision>
+		    <geometry>
+		      <box size="${leglen} 0.1 0.2"/>
+		    </geometry>
+		    <origin xyz="0 0 -${leglen/2}" rpy="0 ${pi/2} 0"/>
+		  </collision>
+		  <xacro:default_inertial mass="10"/>
+		</link>
+		<joint name="base_to_${prefix}_leg" type="fixed">
+		  <parent link="base_link"/>
+		  <child link="${prefix}_leg"/>
+		  <origin xyz="0 ${reflect*(width+.02)} 0.25" />
+		</joint>
+		<link name="${prefix}_base">
+		  <visual>
+		    <geometry>
+		      <box size="${baselen} 0.1 0.1"/>
+		    </geometry>
+		    <material name="white"/>
+		  </visual>
+		  <collision>
+		    <geometry>
+		      <box size="${baselen} 0.1 0.1"/>
+		    </geometry>
+		  </collision>
+		  <xacro:default_inertial mass="10"/>
+		</link>
+		<joint name="${prefix}_base_joint" type="fixed">
+		  <parent link="${prefix}_leg"/>
+		  <child link="${prefix}_base"/>
+		  <origin xyz="0 0 ${-leglen}" />
+		</joint>
+		<xacro:wheel prefix="${prefix}" suffix="front" reflect="1"/>
+		<xacro:wheel prefix="${prefix}" suffix="back" reflect="-1"/>
+	  </xacro:macro>
+	<!--
 	<xacro:macro name="robot_wheel" params="prefix originY">
 		  <link name="${prefix}_leg">
@@ -60,4 +145,4 @@
 			<origin rpy="0 0 0" xyz="-0.133333333333 0 -0.085"/>
 		  </joint>
-	</xacro:macro>
+	</xacro:macro> -->
 </robot>

File: src/project_one/urdf/robot_inertial_essentials.xacro (robot description, xacro)
@@ -1,2 +1,4 @@
+<?xml version="1.0"?>
+<robot xmlns:xacro="http://ros.org/wiki/xacro" name="robot_essentials">
   <xacro:macro name="default_inertial" params="mass">
     <inertial>
@@ -5,2 +7,3 @@
     </inertial>
   </xacro:macro>
+</robot>
